Commit message: added models to gripper urdf

File: gki_cube_gripper_description/urdf/common_properties.urdf.xacro (robot description, xacro)
@@ -5,5 +5,5 @@
 <robot name="xacro_properties" xmlns:xacro="http://ros.org/wiki/xacro">
   <xacro:property name="M_PI" value="3.1415926535897931" />
-  <xacro:property name="M_DEGREE" value="${M_PI/180.0}" />
+  <xacro:property name="M_DEGREES" value="${M_PI/180.0}" />
   <xacro:property name="material_white">
     <material name="white">

File: gki_cube_gripper_description/urdf/cube_gripper.urdf.xacro (robot description, xacro)
@@ -7,15 +7,24 @@
 	<xacro:include filename="$(find gki_cube_gripper_description)/urdf/common_properties.urdf.xacro" />
   <xacro:macro name="cube_gripper" params="name parent *origin">
-    <joint name="${name}_elbow_joint" type="fixed">
+    <joint name="${name}_joint" type="fixed">
       <insert_block name="origin" />
       <parent link="${parent}"/>
-      <child link="${name}_base_link"/>
-    </joint>
-    <joint name="${name}_joint" type="fixed">
-      <origin xyz="0 0 0.056" rpy="0 0 0" />
-      <parent link="${name}_base_link"/>
       <child link="${name}_link"/>
     </joint>
-    <link name="${name}_base_link" />
+    <joint name="${name}_elbow_joint" type="revolute">
+      <axis xyz="0 1 0"/>
+      <limit effort="1000.0" lower="-1.6" upper="0" velocity="0.33"/>
+      <origin xyz="0 0 0" rpy="0 0 0" />
+      <parent link="${name}_link"/>
+      <child link="${name}_arm_link"/>
+    </joint>
+    <joint name="${name}_wrist_joint" type="revolute">
+      <axis xyz="0 0 1"/>
+      <limit effort="1000.0" lower="-1.0" upper="0" velocity="0.33"/>
+      <origin xyz="0 0 0" rpy="0 0 ${90  * M_DEGREES}" />
+      <parent link="${name}_arm_link"/>
+      <child link="${name}_right_finger_link"/>
+    </joint>
+    <link name="${name}_link" />
     <link name="${name}_right_finger_link">
       <inertial>
@@ -27,7 +36,10 @@
         <origin xyz="0 0 0" rpy="0 0 0" />
         <geometry>
+          <!--
+          <box size="0.13 0.13 0.07" />
+          -->
           <mesh filename="package://gki_cube_gripper_description/meshes/cube_gripper_finger.stl"/>
         </geometry>
-        <insert_block name="material_dark_gray" />
+        <xacro:insert_block name="material_dark_grey" />
       </visual>
       <collision>
@@ -47,7 +59,10 @@
         <origin xyz="0 0 0" rpy="0 0 0" />
         <geometry>
+          <!--
+          <box size="0.13 0.13 0.07" />
+          -->
           <mesh filename="package://gki_cube_gripper_description/meshes/cube_gripper_arm.stl"/>
         </geometry>
-        <insert_block name="material_dark_gray" />
+        <xacro:insert_block name="material_dark_grey" />
       </visual>
       <collision>
@@ -58,4 +73,5 @@
       </collision>
     </link>
+<!--
     <link name="${name}_right_elbow_link">
       <inertial>
@@ -69,5 +85,5 @@
           <mesh filename="package://gki_cube_gripper_description/meshes/cube_gripper_elbow.stl"/>
         </geometry>
-        <insert_block name="material_dark_gray" />
+        <xacro:insert_block name="material_dark_grey" />
       </visual>
       <collision>
@@ -81,5 +97,5 @@
       <inertial>
         <mass value="0.200" />
-        <origin xyz="0 0 0" rpy="${180 * M_DEGREE} 0 0" />
+        <origin xyz="0 0 0" rpy="${180 * M_DEGREES} 0 0" />
         <inertia ixx="2.632e-4" ixy="0" ixz="0" iyy="2.632e-4" iyz="0" izz="1.62e-4" />
       </inertial>
@@ -89,5 +105,5 @@
           <mesh filename="package://gki_cube_gripper_description/meshes/cube_gripper_elbow.stl"/>
         </geometry>
-        <insert_block name="material_dark_gray" />
+        <xacro:insert_block name="material_dark_grey" />
       </visual>
       <collision>
@@ -98,4 +114,5 @@
       </collision>
     </link>
+-->
   </xacro:macro>
 </robot>
