Commit message: fixed scale, added correct joint distances

File: gki_cube_gripper_description/urdf/cube_gripper.urdf.xacro (robot description, xacro)
@@ -15,17 +15,24 @@
       <axis xyz="0 1 0"/>
       <limit effort="1000.0" lower="-1.6" upper="0" velocity="0.33"/>
-      <origin xyz="0 0 0" rpy="0 0 0" />
+      <origin xyz="0.03 0 0" rpy="0 0 0" />
       <parent link="${name}_link"/>
       <child link="${name}_arm_link"/>
     </joint>
-    <joint name="${name}_wrist_joint" type="revolute">
+    <joint name="${name}_right_finger_joint" type="revolute">
       <axis xyz="0 0 1"/>
       <limit effort="1000.0" lower="-1.0" upper="0" velocity="0.33"/>
-      <origin xyz="0 0 0" rpy="0 0 ${90  * M_DEGREES}" />
+      <origin xyz="0.175 -0.025 0" rpy="0 0 0" />
       <parent link="${name}_arm_link"/>
       <child link="${name}_right_finger_link"/>
     </joint>
-    <link name="${name}_link" />
-    <link name="${name}_right_finger_link">
+    <joint name="${name}_left_finger_joint" type="revolute">
+      <axis xyz="0 0 1"/>
+      <limit effort="1000.0" lower="-1.0" upper="0" velocity="0.33"/>
+      <origin xyz="0.175 0.025 0" rpy="${180*M_DEGREES} 0 0" />
+      <parent link="${name}_arm_link"/>
+      <child link="${name}_left_finger_link"/>
+      <mimic joint="${name}_right_finger_joint" multiplier="1" />
+    </joint>
+    <link name="${name}_link">
       <inertial>
         <mass value="0.200" />
@@ -36,8 +43,5 @@
         <origin xyz="0 0 0" rpy="0 0 0" />
         <geometry>
-          <!--
-          <box size="0.13 0.13 0.07" />
-          -->
-          <mesh filename="package://gki_cube_gripper_description/meshes/cube_gripper_finger.stl"/>
+          <mesh scale="0.001 0.001 0.001"  filename="package://gki_cube_gripper_description/meshes/cube_gripper_elbow.stl"/>
         </geometry>
         <xacro:insert_block name="material_dark_grey" />
@@ -62,5 +66,51 @@
           <box size="0.13 0.13 0.07" />
           -->
-          <mesh filename="package://gki_cube_gripper_description/meshes/cube_gripper_arm.stl"/>
+          <mesh scale="0.001 0.001 0.001" filename="package://gki_cube_gripper_description/meshes/cube_gripper_arm.stl"/>
+        </geometry>
+        <xacro:insert_block name="material_dark_grey" />
+      </visual>
+      <collision>
+        <origin xyz="0 0 -0.021" rpy="0 0 0" />
+        <geometry>
+          <box size="0.13 0.13 0.07" />
+        </geometry>
+      </collision>
+    </link>
+    <link name="${name}_right_finger_link">
+      <inertial>
+        <mass value="0.200" />
+        <origin xyz="0 0 0" rpy="0 0 0" />
+        <inertia ixx="2.632e-4" ixy="0" ixz="0" iyy="2.632e-4" iyz="0" izz="1.62e-4" />
+      </inertial>
+      <visual>
+        <origin xyz="0 0 0" rpy="0 0 0" />
+        <geometry>
+          <!--
+          <box size="0.13 0.13 0.07" />
+          -->
+          <mesh scale="0.001 0.001 0.001" filename="package://gki_cube_gripper_description/meshes/cube_gripper_finger.stl"/>
+        </geometry>
+        <xacro:insert_block name="material_dark_grey" />
+      </visual>
+      <collision>
+        <origin xyz="0 0 -0.021" rpy="0 0 0" />
+        <geometry>
+          <box size="0.13 0.13 0.07" />
+        </geometry>
+      </collision>
+    </link>
+    <link name="${name}_left_finger_link">
+      <inertial>
+        <mass value="0.200" />
+        <origin xyz="0 0 0" rpy="0 0 0" />
+        <inertia ixx="2.632e-4" ixy="0" ixz="0" iyy="2.632e-4" iyz="0" izz="1.62e-4" />
+      </inertial>
+      <visual>
+        <origin xyz="0 0 0" rpy="0 0 0" />
+        <geometry>
+          <!--
+          <box size="0.13 0.13 0.07" />
+          -->
+          <mesh scale="0.001 0.001 0.001" filename="package://gki_cube_gripper_description/meshes/cube_gripper_finger.stl"/>
         </geometry>
         <xacro:insert_block name="material_dark_grey" />

Commit message: bugfixes in urdf

File: gki_cube_gripper_description/urdf/cube_gripper.urdf.xacro (robot description, xacro)
@@ -14,5 +14,5 @@
     <joint name="${name}_elbow_joint" type="revolute">
       <axis xyz="0 1 0"/>
-      <limit effort="1000.0" lower="-1.6" upper="0" velocity="0.33"/>
+      <limit effort="1000.0" lower="${-90*M_DEGREES}" upper="${90*M_DEGREES}" velocity="0.33"/>
       <origin xyz="0.03 0 0" rpy="0 0 0" />
       <parent link="${name}_link"/>

Commit message: added motor links to get the correct angle offsets

File: gki_cube_gripper_description/urdf/cube_gripper.urdf.xacro (robot description, xacro)
@@ -12,25 +12,41 @@
       <child link="${name}_link"/>
     </joint>
+    <joint name="${name}_lift_motor_joint" type="revolute">
+      <axis xyz="0 1 0"/>
+      <limit effort="1000.0" lower="${-140*M_DEGREES}" upper="${45*M_DEGREES}" velocity="0.33"/>
+      <origin xyz="0.0 0 0" rpy="0 0 0" />
+      <parent link="${name}_link"/>
+      <child link="${name}_lift_motor_link"/>
+    </joint>
+    <joint name="${name}_grab_motor_joint" type="revolute">
+      <axis xyz="0 0 1"/>
+      <limit effort="1000.0" lower="-1.0" upper="0" velocity="1.17"/>
+      <origin xyz="0.0 -0.025 0" rpy="0 0 0" />
+      <parent link="${name}_arm_link"/>
+      <child link="${name}_grab_motor_link"/>
+    </joint>
     <joint name="${name}_elbow_joint" type="revolute">
       <axis xyz="0 1 0"/>
-      <limit effort="1000.0" lower="${-90*M_DEGREES}" upper="${90*M_DEGREES}" velocity="0.33"/>
+      <limit effort="1000.0" lower="${-140*M_DEGREES}" upper="${45*M_DEGREES}" velocity="0.33"/>
       <origin xyz="0.03 0 0" rpy="0 0 0" />
       <parent link="${name}_link"/>
       <child link="${name}_arm_link"/>
+      <mimic joint="${name}_lift_motor_joint" multiplier="-1" offset="${-50*M_DEGREES}"/>
     </joint>
     <joint name="${name}_right_finger_joint" type="revolute">
       <axis xyz="0 0 1"/>
-      <limit effort="1000.0" lower="-1.0" upper="0" velocity="0.33"/>
+      <limit effort="1000.0" lower="-1.0" upper="0" velocity="1.17"/>
       <origin xyz="0.175 -0.025 0" rpy="0 0 0" />
       <parent link="${name}_arm_link"/>
       <child link="${name}_right_finger_link"/>
+      <mimic joint="${name}_grab_motor_joint" multiplier="-1" offset="${-55*M_DEGREES}"/>
     </joint>
     <joint name="${name}_left_finger_joint" type="revolute">
       <axis xyz="0 0 1"/>
-      <limit effort="1000.0" lower="-1.0" upper="0" velocity="0.33"/>
+      <limit effort="1000.0" lower="-1.0" upper="0" velocity="1.17"/>
       <origin xyz="0.175 0.025 0" rpy="${180*M_DEGREES} 0 0" />
       <parent link="${name}_arm_link"/>
       <child link="${name}_left_finger_link"/>
-      <mimic joint="${name}_right_finger_joint" multiplier="1" />
+      <mimic joint="${name}_grab_motor_joint" multiplier="-1" offset="${-55*M_DEGREES}"/>
     </joint>
     <link name="${name}_link">
@@ -123,46 +139,6 @@
       </collision>
     </link>
-<!--
-    <link name="${name}_right_elbow_link">
-      <inertial>
-        <mass value="0.200" />
-        <origin xyz="0 0 0" rpy="0 0 0" />
-        <inertia ixx="2.632e-4" ixy="0" ixz="0" iyy="2.632e-4" iyz="0" izz="1.62e-4" />
-      </inertial>
-      <visual>
-        <origin xyz="0 0 0" rpy="0 0 0" />
-        <geometry>
-          <mesh filename="package://gki_cube_gripper_description/meshes/cube_gripper_elbow.stl"/>
-        </geometry>
-        <xacro:insert_block name="material_dark_grey" />
-      </visual>
-      <collision>
-        <origin xyz="0 0 -0.021" rpy="0 0 0" />
-        <geometry>
-          <box size="0.13 0.13 0.07" />
-        </geometry>
-      </collision>
-    </link>
-    <link name="${name}_left_elbow_link">
-      <inertial>
-        <mass value="0.200" />
-        <origin xyz="0 0 0" rpy="${180 * M_DEGREES} 0 0" />
-        <inertia ixx="2.632e-4" ixy="0" ixz="0" iyy="2.632e-4" iyz="0" izz="1.62e-4" />
-      </inertial>
-      <visual>
-        <origin xyz="0 0 0" rpy="0 0 0" />
-        <geometry>
-          <mesh filename="package://gki_cube_gripper_description/meshes/cube_gripper_elbow.stl"/>
-        </geometry>
-        <xacro:insert_block name="material_dark_grey" />
-      </visual>
-      <collision>
-        <origin xyz="0 0 -0.021" rpy="0 0 0" />
-        <geometry>
-          <box size="0.13 0.13 0.07" />
-        </geometry>
-      </collision>
-    </link>
--->
+    <link name="${name}_grab_motor_link"/>
+    <link name="${name}_lift_motor_link"/>
   </xacro:macro>
 </robot>

Commit message: corrected collision model

File: gki_cube_gripper_description/urdf/cube_gripper.urdf.xacro (robot description, xacro)
@@ -102,7 +102,4 @@
         <origin xyz="0 0 0" rpy="0 0 0" />
         <geometry>
-          <!--
-          <box size="0.13 0.13 0.07" />
-          -->
           <mesh scale="0.001 0.001 0.001" filename="package://gki_cube_gripper_description/meshes/cube_gripper_finger.stl"/>
         </geometry>
@@ -110,7 +107,7 @@
       </visual>
       <collision>
-        <origin xyz="0 0 -0.021" rpy="0 0 0" />
+        <origin xyz="0.1 -0.05 0" rpy="0 0 0" />
         <geometry>
-          <box size="0.13 0.13 0.07" />
+          <box size="0.2 0.1 0.05" />
         </geometry>
       </collision>
@@ -133,7 +130,7 @@
       </visual>
       <collision>
-        <origin xyz="0 0 -0.021" rpy="0 0 0" />
+        <origin xyz="0.1 -0.05 0" rpy="0 0 0" />
         <geometry>
-          <box size="0.13 0.13 0.07" />
+          <box size="0.2 0.1 0.05" />
         </geometry>
       </collision>
